Commit message: simulate in gazebo

File: description/robot_core.xacro (robot description, xacro)
@@ -38,4 +38,9 @@
         </xacro:inertial_box>
     </link>
+    <gazebo reference="chassis">
+    <material>
+        Gazebo/Blue
+    </material>
+    </gazebo>
     <joint name="left_wheel_joint" type="continuous">
         <parent link="base_link"/>
@@ -59,4 +64,9 @@
         </xacro:inertial_cylinder>
     </link>
+    <gazebo reference="left_wheel">
+    <material>
+        Gazebo/Black
+    </material>
+    </gazebo>
     <joint name="right_wheel_joint" type="continuous">
         <parent link="base_link"/>
@@ -80,4 +90,9 @@
         </xacro:inertial_cylinder>
     </link>
+    <gazebo reference="right_wheel">
+    <material>
+        Gazebo/Black
+    </material>
+    </gazebo>
         <!-- CASTER WHEEL -->
     <joint name="caster_wheel_joint" type="fixed">
@@ -102,3 +117,10 @@
         </xacro:inertial_sphere>
     </link>
+    <gazebo reference="caster_wheel">
+    <material>
+        Gazebo/Brown
+    </material>
+    <mu1 value="0.001"/>
+    <mu2 value="0.001"/>
+    </gazebo>
 </robot>
